File: eagle design files/AEMSUCA-R2.brd (EAGLE design)
At the start: 20.3 x 15.2 mm, 16 parts, among them IC1 AEM10941, Q1 DMG1012UW

Commit message: updated PCB and gerbers to reduce solderpaste under IC1 to 50%
Parts:
- IC1: device sodaq:QFN50P505X505X90-28 -> TSEM:QFN50P505X505X90-28
Changed lines of the file:
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@@
 <layer number="29" name="tStop" color="7" fill="3" visible="no" active="yes"/>
 <layer number="30" name="bStop" color="7" fill="6" visible="no" active="yes"/>
-<layer number="31" name="tCream" color="7" fill="4" visible="no" active="yes"/>
+<layer number="31" name="tCream" color="7" fill="4" visible="yes" active="yes"/>
 <layer number="32" name="bCream" color="7" fill="5" visible="no" active="yes"/>
 <layer number="33" name="tFinish" color="6" fill="3" visible="no" active="yes"/>
@@
 </autorouter>
 <elements>
-<element name="IC1" library="sodaq" package="QFN50P505X505X90-28" package3d_urn="urn:adsk.eagle:package:2265650/1" value="AEM10941" x="10.7" y="7.3" smashed="yes" rot="R90">
+<element name="IC1" library="TSEM" package="QFN50P505X505X90-28" value="AEM10941" x="10.7" y="7.3" smashed="yes" rot="R90">
 <attribute name="MF" value="e-peas" x="10.7" y="7.3" size="1.778" layer="27" rot="R90" display="off"/>
 <attribute name="MPN" value="AEM10941" x="10.7" y="7.3" size="1.778" layer="27" rot="R90" display="off"/>
@@
 which will not be processed correctly with this version.
 </note>
-<note version="8.3" severity="warning">
-Since Version 8.3, EAGLE supports URNs for individual library
-assets (packages, symbols, and devices). The URNs of those assets
-will not be understood (or retained) with this version.
-</note>
-<note version="8.3" severity="warning">
-Since Version 8.3, EAGLE supports the association of 3D packages
-with devices in libraries, schematics, and board files. Those 3D
-packages will not be understood (or retained) with this version.
-</note>
 </compatibility>
